Commit message: Refactoring

File: src/amiga_nav2/urdf/amiga.urdf (robot description, URDF)
Before this commit: robot amiga_robot, 7 links, 6 joints
Links:
- link base_link: geometry visual mesh filename=package://amiga_nav2/meshes/amiga_body.stl scale=0.001 0.001 0.001
- link front_left_wheel: geometry visual mesh filename=package://amiga_nav2/meshes/amiga_wheel.stl scale=0.001 0.001 0.001
- link front_right_wheel: geometry visual mesh filename=package://amiga_nav2/meshes/amiga_wheel.stl scale=0.001 0.001 0.001
- link rear_left_wheel: geometry visual mesh filename=package://amiga_nav2/meshes/amiga_wheel.stl scale=0.001 0.001 0.001
- link rear_right_wheel: geometry visual mesh filename=package://amiga_nav2/meshes/amiga_wheel.stl scale=0.001 0.001 0.001
